Commit message: Actualizo phantom_ws con cambios

File: Codigos/phantom_ws/install/phantomx_pincher_description/share/phantomx_pincher_description/urdf/kit.xacro (robot description, xacro)
@@ -62,4 +62,69 @@
     <child link="caseBaseRobot_link" />
     <origin xyz="-0.01325 0 0.054" rpy="0 0 0" />
+  </joint>
+  <link name="canastilla_link">
+    <visual>
+      <origin xyz="0.155 0 0" rpy="0 0 0" />
+      <geometry>
+        <mesh filename="package://phantomx_pincher_description/meshes/STL/canastilla.stl"
+              scale="0.001 0.001 0.001" />
+      </geometry>
+      <material name="blue" />
+    </visual>
+    <collision>
+        <origin xyz="-0.1365 0.0 0.0905" rpy="0 0 0" />
+        <geometry>
+            <box size="0.017 0.4 0.1855" />
+        </geometry>
+        <material name="blue" />
+    </collision>
+    <collision>
+        <origin xyz="0.4465 0.0 0.0905" rpy="0 0 0" />
+        <geometry>
+            <box size="0.017 0.4 0.1855" />
+        </geometry>
+        <material name="blue" />
+    </collision>
+    <collision>
+        <origin xyz="0.155 0.1915 0.0905" rpy="0 0 0" />
+        <geometry>
+            <box size="0.6 0.017 0.1855" />
+        </geometry>
+        <material name="blue" />
+    </collision>
+    <collision>
+        <origin xyz="0.155 -0.1915 0.0905" rpy="0 0 0" />
+        <geometry>
+            <box size="0.6 0.017 0.1855" />
+        </geometry>
+        <material name="blue" />
+    </collision>
+  </link>
+  <joint name="base_canastilla_joint" type="fixed">
+    <parent link="baseFija_link" />
+    <child link="canastilla_link" />
+    <origin xyz="0 0 0" rpy="0 0 0" />
+  </joint>
+  <link name="ensambleSoporteCamara_link">
+    <visual>
+      <origin xyz="0.26028 0 0" rpy="0 0 -${PI/2}" />
+      <geometry>
+        <mesh filename="package://phantomx_pincher_description/meshes/STL/ensambleSoporteCamara.stl"
+              scale="0.001 0.001 0.001" />
+      </geometry>
+      <material name="gray" />
+    </visual>
+    <collision>
+        <origin xyz="0.26028 0 0.08508" rpy="0 0 -${PI/2}" />
+        <geometry>
+            <box size="0.04 0.025 0.17016" />
+        </geometry>
+        <material name="gray" />
+    </collision>
+  </link>
+  <joint name="base_ensambleSoporteCamara_joint" type="fixed">
+    <parent link="baseFija_link" />
+    <child link="ensambleSoporteCamara_link" />
+    <origin xyz="0 0 0" rpy="0 0 0" />
   </joint>
   <link name="zonaRecoleccion_link">
